Commit message: add new impedance controller

File: advanced-robotics/elfin/elfin_description/urdf/camera_world.xacro (robot description, xacro)
@@ -1,17 +1,17 @@
 <?xml version="1.0"?>
 <robot xmlns:xacro="http://www.ros.org/wiki/xacro">
-  <xacro:property name="camera_link" value="0.03" /> <!-- Size of square 'camera' box -->
+  <xacro:property name="camera_link_world" value="0.03" /> <!-- Size of square 'camera' box -->
   <xacro:property name="PI" value="3.1415926535897931"/>
-  <link name="camera_link">
+  <link name="camera_link_world">
     <collision>
-      <origin xyz="0.0 0.0 0.00" rpy="0 0 0.0"/>
+      <origin xyz="0.0 0.0 0.0" rpy="0 0 0.0"/>
       <geometry>
-    <box size="${camera_link} ${camera_link} ${camera_link}"/>
+    <box size="${camera_link_world} ${camera_link_world} ${camera_link_world}"/>
       </geometry>
     </collision>
     <visual>
-      <origin xyz="0 0 0.00" rpy="0 0 0"/>
+      <origin xyz="0.0 0.0 0.0" rpy="0 0 0"/>
       <geometry>
-    <box size="${camera_link} ${camera_link} ${camera_link}"/>
+    <box size="${camera_link_world} ${camera_link_world} ${camera_link_world}"/>
       </geometry>
       <material name="red"/>
@@ -23,21 +23,21 @@
     </inertial>
   </link>
- <joint name="camera_joint" type="fixed">
-    <axis xyz="0 1 0" />
-    <origin xyz="0 0.00 -0.03" rpy="${PI} ${-PI/2} 0"/>
-    <parent link="elfin_dummy_gripper"/>
-    <child link="camera_link"/>
+ <joint name="camera_joint_world" type="fixed">
+    <axis xyz="0.0 0 0" />
+    <origin xyz="0.0 0.00 2.0" rpy="0 ${PI/2} 0"/>
+    <parent link="world"/>
+    <child link="camera_link_world"/>
   </joint>
-  <link name="camera_link_optical">
+  <link name="camera_link_world_optical">
   </link>
-  <joint name="camera_optical_joint" type="fixed">
+  <joint name="camera_optical_joint_world" type="fixed">
     <!-- these values have to be these values otherwise the gazebo camera
         image won't be aligned properly with the frame it is supposedly
         originating from -->
-    <origin xyz="0 0 0" rpy="${-pi/2} 0 ${-pi/2}"/>
-    <parent link="camera_link"/>
-    <child link="camera_link_optical"/>
+    <origin xyz="0.0 0 0.0" rpy="0.0 ${PI/2} 0.0"/>
+    <parent link="camera_link_world"/>
+    <child link="camera_link_world_optical"/>
   </joint>
-<gazebo reference="camera_link">
+<gazebo reference="camera_link_world">
   <sensor name="camera" type="depth">
     <update_rate>20</update_rate>
@@ -64,5 +64,5 @@
       <depthImageInfoTopicName>/camera/depth/camera_info</depthImageInfoTopicName>
       <pointCloudTopicName>/camera/depth/points</pointCloudTopicName>
-      <frameName>camera_link_optical</frameName>
+      <frameName>camera_link_world_optical</frameName>
       <pointCloudCutoff>0.5</pointCloudCutoff>
       <pointCloudCutoffMax>3.0</pointCloudCutoffMax>

File: advanced-robotics/elfin/elfin_description/urdf/elfin3.urdf.xacro (robot description, xacro)
@@ -1,7 +1,4 @@
 <robot
   name="elfin3" xmlns:xacro="http://www.ros.org/wiki/xacro">
-  <xacro:include filename="$(find elfin_description)/urdf/materials.xacro" />
-  <xacro:include filename="$(find elfin_description)/urdf/elfin_robot.gazebo" />
-  <xacro:include filename="$(find elfin_description)/urdf/elfin_transmission.xacro" />
   <xacro:property name="PI" value="3.1415926535897931"/>
   <link name="world"/>
@@ -430,3 +427,7 @@
       link="elfin_dummy_gripper" />
   </joint>
+  <xacro:include filename="$(find elfin_description)/urdf/materials.xacro" />
+  <xacro:include filename="$(find elfin_description)/urdf/elfin_robot.gazebo" />
+  <xacro:include filename="$(find elfin_description)/urdf/elfin_transmission.xacro" />
+  <xacro:include filename="$(find elfin_description)/urdf/camera_world.xacro" />
 </robot>

Commit message: add files for the final check => tag follower, voice commands, launch configuration

File: advanced-robotics/elfin/elfin_description/urdf/camera_world.xacro (robot description, xacro)
@@ -25,5 +25,5 @@
  <joint name="camera_joint_world" type="fixed">
     <axis xyz="0.0 0 0" />
-    <origin xyz="0.0 0.00 2.0" rpy="0 ${PI/2} 0"/>
+    <origin xyz="0.0 0.00 1.5" rpy="0.0 ${PI/2} 0.0"/>
     <parent link="world"/>
     <child link="camera_link_world"/>
@@ -35,5 +35,5 @@
         image won't be aligned properly with the frame it is supposedly
         originating from -->
-    <origin xyz="0.0 0 0.0" rpy="0.0 ${PI/2} 0.0"/>
+    <origin xyz="0.0 0 0.0" rpy="-${PI/2} 0.0 -${PI/2}"/>
     <parent link="camera_link_world"/>
     <child link="camera_link_world_optical"/>
@@ -41,5 +41,5 @@
 <gazebo reference="camera_link_world">
   <sensor name="camera" type="depth">
-    <update_rate>20</update_rate>
+    <update_rate>10</update_rate>
     <camera>
       <horizontal_fov>1.047198</horizontal_fov>
@@ -59,6 +59,6 @@
       <updateRate>1.0</updateRate>
       <cameraName></cameraName>
-      <imageTopicName>/camera/image</imageTopicName>
-      <cameraInfoTopicName>/camera/camera_info</cameraInfoTopicName>
+      <imageTopicName>/camera/image/world</imageTopicName>
+      <cameraInfoTopicName>/camera/camera_info/world</cameraInfoTopicName>
       <depthImageTopicName>/camera/depth/image_raw</depthImageTopicName>
       <depthImageInfoTopicName>/camera/depth/camera_info</depthImageInfoTopicName>

File: advanced-robotics/elfin/elfin_description/urdf/elfin3.urdf.xacro (robot description, xacro)
@@ -431,3 +431,4 @@
   <xacro:include filename="$(find elfin_description)/urdf/elfin_transmission.xacro" />
   <xacro:include filename="$(find elfin_description)/urdf/camera_world.xacro" />
+  <xacro:include filename="$(find elfin_description)/urdf/camera.xacro" />
 </robot>
