Commit message: Working

File: advanced-robotics/elfin/elfin_description/urdf/elfin3.urdf.xacro (robot description, xacro)
@@ -410,23 +410,81 @@
       velocity="1.57" />
   </joint>
-  <link name="elfin_end_link"/>
-  <joint name="elfin_end_joint" type="fixed">
-    <origin
-      xyz="0 -0.091 0"
-      rpy="${PI/2} ${-PI/2} 0" />
-    <parent
-      link="elfin_link6" />
-    <child
-      link="elfin_end_link" />
-  </joint>
-  <link name="elfin_dummy_gripper"/>
-  <joint name="elfin_dummy_joint" type="fixed">
-    <origin
-      xyz="0 -0.111 0"
-      rpy="${PI/2} ${-PI/2} 0" />
-    <parent
-      link="elfin_link6" />
-    <child
-      link="elfin_dummy_gripper" />
+  <link name="elfin_tool">
+    <collision>
+      <origin xyz="0 0 0" rpy="${PI/2} 0 0"/>
+      <geometry>
+        <cylinder length="0.08" radius="0.01"/>
+      </geometry>
+    </collision>
+    <visual>
+      <origin xyz="0 0 0" rpy="${PI/2} 0 0" />
+      <geometry>
+        <cylinder length="0.08" radius="0.01"/>
+      </geometry>
+    </visual>
+    <inertial>
+      <mass value="0.01" />
+      <origin xyz="0 0 0" rpy="0 0 0"/>
+      <inertia ixx="0.01" ixy="0" ixz="0" iyy="0.01" iyz="0" izz="0.01" />
+    </inertial>
+  </link>
+  <joint name="tool_joint" type="fixed">
+    <parent link="elfin_link6"/>
+    <child link="elfin_tool"/>
+    <origin xyz="0 -0.08 0" rpy="0 0 0" />
+  </joint>
+  <link name="elfin_ft_sensor_link">
+    <collision>
+      <origin xyz="0 0 0" rpy="${PI/2} 0 0"/>
+      <geometry>
+        <cylinder length="0.02" radius="0.01"/>
+      </geometry>
+    </collision>
+    <visual>
+      <origin xyz="0 0 0" rpy="${PI/2} 0 0" />
+      <geometry>
+        <cylinder length="0.02" radius="0.01"/>
+      </geometry>
+    </visual>
+    <inertial>
+      <mass value="0.01" />
+      <origin xyz="0 0 0" rpy="0 0 0"/>
+      <inertia ixx="0.01" ixy="0" ixz="0" iyy="0.01" iyz="0" izz="0.01" />
+    </inertial>
+  </link>
+  <joint name="ft_sensor_joint" type="revolute">
+    <parent link="elfin_tool"/>
+    <child link="elfin_ft_sensor_link"/>
+    <origin xyz="0 -0.02 0" rpy="0 0 0" />
+    <axis xyz="0 -1 0"/>
+    <limit
+      lower="0.0"
+      upper="0.0"
+      effort="0.0"
+      velocity="0.0" />
+  </joint>
+  <link name="elfin_tool_ball">
+    <collision>
+      <origin xyz="0 0 0" rpy="0 0 0"/>
+      <geometry>
+        <sphere radius="0.02"/>
+      </geometry>
+    </collision>
+    <visual>
+      <origin xyz="0 0 0" rpy="0 0 0" />
+      <geometry>
+        <sphere radius="0.02"/>
+      </geometry>
+    </visual>
+    <inertial>
+      <mass value="0.01" />
+      <origin xyz="0 0 0" rpy="0 0 0"/>
+      <inertia ixx="0.01" ixy="0" ixz="0" iyy="0.01" iyz="0" izz="0.01" />
+    </inertial>
+  </link>
+  <joint name="tool_ball_joint" type="fixed">
+    <parent link="elfin_tool"/>
+    <child link="elfin_tool_ball"/>
+    <origin xyz="0 -0.04 0" rpy="0 0 0" />
   </joint>
 </robot>

File: advanced-robotics/elfin/elfin_description/urdf/elfin_transmission.xacro (robot description, xacro)
@@ -56,3 +56,12 @@
       </actuator>
     </transmission>
+    <transmission name="elfin_joint7_trans">
+      <type>transmission_interface/SimpleTransmission</type>
+      <joint name="ft_sensor_joint">
+        <hardwareInterface>hardware_interface/EffortJointInterface</hardwareInterface>
+      </joint>
+      <actuator name="ft_sensor_joint_motor">
+        <mechanicalReduction>1</mechanicalReduction>
+      </actuator>
+    </transmission>
 </robot>

Commit message: before solving the inverse kinematic

File: advanced-robotics/elfin/elfin_description/urdf/elfin3.urdf.xacro (robot description, xacro)
@@ -458,11 +458,38 @@
     <origin xyz="0 -0.02 0" rpy="0 0 0" />
     <axis xyz="0 -1 0"/>
-    <limit
-      lower="0.0"
-      upper="0.0"
+    <dynamics
+      damping="10"
+      spring="100"
+      friction="1" />
+    <limit
+      lower="0.01"
+      upper="0.01"
       effort="0.0"
       velocity="0.0" />
   </joint>
   <link name="elfin_tool_ball">
+    <collision>
+      <origin xyz="0 0 0" rpy="0 0 0"/>
+      <geometry>
+        <sphere radius="0.02"/>
+      </geometry>
+      <surface>
+        <friction>
+          <ode>
+            <mu>0.01</mu>
+            <mu2>0.01</mu2>
+            <fdir1>0 0 1</fdir1>
+            <slip1>0.0</slip1>
+            <slip2>0.0</slip2>
+          </ode>
+        </friction>
+        <contact>
+          <ode>
+            <min_depth>5</min_depth>
+            <kp>1e6</kp>
+          </ode>
+        </contact>
+      </surface>
+    </collision>
     <collision>
       <origin xyz="0 0 0" rpy="0 0 0"/>

File: advanced-robotics/elfin/elfin_description/urdf/my_box.urdf.xacro (robot description, xacro)
@@ -35,4 +35,21 @@
          <box size="0.1 1 1"/>
       </geometry>
+      <surface>
+        <friction>
+          <ode>
+            <mu>0.01</mu>
+            <mu2>0.01</mu2>
+            <fdir1>0 0 1</fdir1>
+            <slip1>0.0</slip1>
+            <slip2>0.0</slip2>
+          </ode>
+        </friction>
+        <contact>
+          <ode>
+            <min_depth>5</min_depth>
+            <kp>1e6</kp>
+          </ode>
+        </contact>
+      </surface>
     </collision>
     <inertial>
