Commit message: Add needed files for tag detection and tag following

File: advanced-robotics/elfin/elfin_description/urdf/camera.xacro (robot description, xacro)
@@ -1,8 +1,9 @@
 <?xml version="1.0"?>
 <robot xmlns:xacro="http://www.ros.org/wiki/xacro">
-  <xacro:property name="camera_link" value="0.05" /> <!-- Size of square 'camera' box -->
+  <xacro:property name="camera_link" value="0.03" /> <!-- Size of square 'camera' box -->
+  <xacro:property name="PI" value="3.1415926535897931"/>
   <link name="camera_link">
     <collision>
-      <origin xyz="0 0 0" rpy="0 0 0"/>
+      <origin xyz="0.0 0.0 0.00" rpy="0 0 0.0"/>
       <geometry>
     <box size="${camera_link} ${camera_link} ${camera_link}"/>
@@ -10,5 +11,5 @@
     </collision>
     <visual>
-      <origin xyz="0 0 0" rpy="0 0 0"/>
+      <origin xyz="0 0 0.00" rpy="0 0 0"/>
       <geometry>
     <box size="${camera_link} ${camera_link} ${camera_link}"/>
@@ -24,46 +25,58 @@
  <joint name="camera_joint" type="fixed">
     <axis xyz="0 1 0" />
-    <origin xyz="0.0 0 -0.08" rpy="0 0 -1.57"/>
-    <parent link="elfin_link6"/>
+    <origin xyz="0 0.05 -0.02" rpy="${PI} ${-PI/2} 0"/>
+    <parent link="elfin_dummy_gripper"/>
     <child link="camera_link"/>
   </joint>
-  <gazebo reference="camera_link">
-    <sensor type="camera" name="camera1">
-      <update_rate>30.0</update_rate>
-      <camera name="head">
-        <horizontal_fov>1.3962634</horizontal_fov>
-        <image>
-          <width>800</width>
-          <height>800</height>
-          <format>R8G8B8</format>
-        </image>
-        <clip>
-          <near>0.02</near>
-          <far>300</far>
-        </clip>
-        <noise>
-          <type>gaussian</type>
-          <!-- Noise is sampled independently per pixel on each frame.
-               That pixel's noise value is added to each of its color
-               channels, which at that point lie in the range [0,1]. -->
-          <mean>0.0</mean>
-          <stddev>0.007</stddev>
-        </noise>
-      </camera>
-      <plugin name="camera_controller" filename="libgazebo_ros_camera.so">
-        <alwaysOn>true</alwaysOn>
-        <updateRate>0.0</updateRate>
-        <cameraName>rrbot/camera1</cameraName>
-        <imageTopicName>image_raw</imageTopicName>
-        <cameraInfoTopicName>camera_info</cameraInfoTopicName>
-        <frameName>camera_link</frameName>
-        <hackBaseline>0.07</hackBaseline>
-        <distortionK1>0.0</distortionK1>
-        <distortionK2>0.0</distortionK2>
-        <distortionK3>0.0</distortionK3>
-        <distortionT1>0.0</distortionT1>
-        <distortionT2>0.0</distortionT2>
-      </plugin>
-    </sensor>
-  </gazebo>
+  <link name="camera_link_optical">
+  </link>
+  <joint name="camera_optical_joint" type="fixed">
+    <!-- these values have to be these values otherwise the gazebo camera
+        image won't be aligned properly with the frame it is supposedly
+        originating from -->
+    <origin xyz="0 0 0" rpy="${-pi/2} 0 ${-pi/2}"/>
+    <parent link="camera_link"/>
+    <child link="camera_link_optical"/>
+  </joint>
+<gazebo reference="camera_link">
+  <sensor name="camera" type="depth">
+    <update_rate>20</update_rate>
+    <camera>
+      <horizontal_fov>1.047198</horizontal_fov>
+      <image>
+        <width>640</width>
+        <height>480</height>
+        <format>R8G8B8</format>
+      </image>
+      <clip>
+        <near>0.05</near>
+        <far>3</far>
+      </clip>
+    </camera>
+    <plugin name="camera_controller" filename="libgazebo_ros_openni_kinect.so">
+      <baseline>0.2</baseline>
+      <alwaysOn>true</alwaysOn>
+      <updateRate>1.0</updateRate>
+      <cameraName></cameraName>
+      <imageTopicName>/camera/image</imageTopicName>
+      <cameraInfoTopicName>/camera/camera_info</cameraInfoTopicName>
+      <depthImageTopicName>/camera/depth/image_raw</depthImageTopicName>
+      <depthImageInfoTopicName>/camera/depth/camera_info</depthImageInfoTopicName>
+      <pointCloudTopicName>/camera/depth/points</pointCloudTopicName>
+      <frameName>camera_link_optical</frameName>
+      <pointCloudCutoff>0.5</pointCloudCutoff>
+      <pointCloudCutoffMax>3.0</pointCloudCutoffMax>
+      <distortionK1>0.00000001</distortionK1>
+      <distortionK2>0.00000001</distortionK2>
+      <distortionK3>0.00000001</distortionK3>
+      <distortionT1>0.00000001</distortionT1>
+      <distortionT2>0.00000001</distortionT2>
+      <CxPrime>0</CxPrime>
+      <Cx>0</Cx>
+      <Cy>0</Cy>
+      <focalLength>0</focalLength>
+      <hackBaseline>0</hackBaseline>
+    </plugin>
+  </sensor>
+</gazebo>
 </robot>

Commit message: Add error print statements and some other debugging tools

File: advanced-robotics/elfin/elfin_description/urdf/camera.xacro (robot description, xacro)
@@ -25,5 +25,5 @@
  <joint name="camera_joint" type="fixed">
     <axis xyz="0 1 0" />
-    <origin xyz="0 0.05 -0.02" rpy="${PI} ${-PI/2} 0"/>
+    <origin xyz="0 0.00 -0.03" rpy="${PI} ${-PI/2} 0"/>
     <parent link="elfin_dummy_gripper"/>
     <child link="camera_link"/>

Commit message: Camera and Admitance Control seems to be working.

File: advanced-robotics/elfin/elfin_description/urdf/camera.xacro (robot description, xacro)
@@ -25,6 +25,6 @@
  <joint name="camera_joint" type="fixed">
     <axis xyz="0 1 0" />
-    <origin xyz="0 0.00 -0.03" rpy="${PI} ${-PI/2} 0"/>
-    <parent link="elfin_dummy_gripper"/>
+    <origin xyz="0 0.00 -0.03" rpy="0 0 ${-PI/2}"/>
+    <parent link="elfin_tool_ball"/>
     <child link="camera_link"/>
   </joint>
@@ -41,5 +41,5 @@
 <gazebo reference="camera_link">
   <sensor name="camera" type="depth">
-    <update_rate>1000</update_rate>
+    <update_rate>20</update_rate>
     <camera>
       <horizontal_fov>1.047198</horizontal_fov>

File: advanced-robotics/elfin/elfin_description/urdf/elfin3.urdf.xacro (robot description, xacro)
@@ -515,3 +515,4 @@
     <origin xyz="0 -0.04 0" rpy="0 0 0" />
   </joint>
+  <xacro:include filename="$(find elfin_description)/urdf/camera.xacro" />
 </robot>
